File: Hardware (kicad)/MPCBoard/MPCBoard.kicad_sch (KiCad schematic)
At the start: 110 parts, among them J1 62000421821, J2 62000421821, J3 62000421821, J4 62000421821, J5 62000421821, J6 62000421821, J7 62000421821, J8 62000421821, P1 61300611121, U1 TS914, U10 PCA9535A, U11 ADS1015IDGST, U12 ADS1015IDGST, U2 TS914, U3 TS914, U4 TS914, U5 TS914, U6 TS914, U7 TS914, U8 TS914

Commit message: fix kicad projects
Parts:
- removed unit 1 of U10
- added unit 2 of U1
- added unit 1 of U10
- added unit 2 of U2
- added unit 2 of U3
- added unit 2 of U4
- added unit 2 of U5
- added unit 2 of U6
- added unit 2 of U7
- added unit 2 of U8
- C1, C11, C21, C31, C41, C51, C61, C71: footprint CAPC0603(1608)100_N -> Capacitor_SMD:C_0603_1608Metric_Pad1.08x0.95mm_HandSolder; symbol Passive SMD:root_1_CAP_Passive SMD.IntLib -> Device:C
- C100, C101, C102, C12, C2, C22, C32, C42, C52, C62, C72: footprint CAPC0603(1608)100_N -> Capacitor_SMD:C_0603_1608Metric_Pad1.08x0.95mm_HandSolder; symbol Passive SMD:root_0_CAP_Passive SMD.IntLib -> Device:C
- J1, J2, J3, J4, J5, J6, J7, J8: footprint 62000421821 -> Wurth_WR-PHD (rev24a):62000421821; symbol Wurth_WR-PHD (rev24a):root_0_62000421821_Wurth_WR-PHD (rev24a).IntLib -> Connector_Generic:Conn_02x02_Odd_Even
- P1: footprint 61300611121 -> Wurth_WR-PHD (rev24a):61300611121; symbol Wurth_WR-PHD (rev24a):root_0_61300611121_Wurth_WR-PHD (rev24a).IntLib -> Connector_Generic:Conn_01x06
- R1, R103, R104, R105, R106, R11, R12, R13, R2, R21, R22, R23, R3, R31, R32, R33, R41, R42, R43, R51, R52, R53, R61, R62, R63, R71, R72, R73: footprint RESC0603(1608)_N -> Resistor_SMD:R_0603_1608Metric_Pad0.98x0.95mm_HandSolder; symbol Passive SMD:root_1_RES_Passive SMD.IntLib -> Device:R_US
- R100, R14, R16, R24, R26, R34, R36, R4, R44, R46, R54, R56, R6, R64, R66, R74, R76: footprint RESC0603(1608)_N -> Resistor_SMD:R_0603_1608Metric_Pad0.98x0.95mm_HandSolder; symbol Passive SMD:root_2_RES_Passive SMD.IntLib -> Device:R_US
- R101, R102, R15, R18, R25, R28, R35, R38, R45, R48, R5, R55, R58, R65, R68, R75, R78, R8: footprint RESC0603(1608)_N -> Resistor_SMD:R_0603_1608Metric_Pad0.98x0.95mm_HandSolder; symbol Passive SMD:root_0_RES_Passive SMD.IntLib -> Device:R_US
- R17, R27, R37, R47, R57, R67, R7, R77: footprint RESC0603(1608)_N -> Resistor_SMD:R_0603_1608Metric_Pad0.98x0.95mm_HandSolder; symbol Passive SMD:root_3_RES_Passive SMD.IntLib -> Device:R_US
- U1, U2, U3, U4, U5, U6, U7, U8: footprint SO-14_STM -> Sampler:TS914IDT; symbol TS914AIDT:root_0_TS914_TS914AIDT.IntLib -> Sampler:TS914IDT
- U10: footprint TSSOP24-8N -> NXP:TSSOP24-8N; symbol NXP:root_0_PCA9535A_NXP.IntLib -> NXP:PCA9535A
- U11, U12: footprint DGS0010A_N -> ADS1015IDGST:SOP50P490X110-10N; symbol ADS1015IDGST:root_0_ADS1015IDGST_ADS1015IDGST.IntLib -> ul_ADS1015IDGST:ADS1015IDGST
Connections:
- net +5V: now also R101.2, R102.2, U10.24 (VDD); no longer R101.1, R102.1
- net BTN_01+: now also C1.1; no longer C1.2
- net BTN_01_OUT: now also R8.2; no longer R8.1
- net BTN_02+: now also C11.1; no longer C11.2
- net BTN_02_OUT: now also R18.2; no longer R18.1
- net BTN_03+: now also C21.1; no longer C21.2
- net BTN_03_OUT: now also R28.2; no longer R28.1
- net BTN_04+: now also C31.1; no longer C31.2
- net BTN_04_OUT: now also R38.2; no longer R38.1
- net BTN_05+: now also C41.1; no longer C41.2
- net BTN_05_OUT: now also R48.2; no longer R48.1
- net BTN_06+: now also C51.1; no longer C51.2
- net BTN_06_OUT: now also R58.2; no longer R58.1
- net BTN_07+: now also C61.1; no longer C61.2
- net BTN_07_OUT: now also R68.2; no longer R68.1
- net BTN_08+: now also C71.1; no longer C71.2
- net BTN_08_OUT: now also R78.2; no longer R78.1
- net GND: now also C1.2, C11.2, C21.2, C31.2, C41.2, C51.2, C61.2, C71.2, R17.2, R27.2, R37.2, R47.2, R57.2, R67.2, R7.2, R77.2, U10.12 (VSS), U10.2 (A1), U10.21 (A0), U10.3 (A2); no longer C1.1, C11.1, C21.1, C31.1, C41.1, C51.1, C61.1, C71.1, R17.1, R27.1, R37.1, R47.1, R57.1, R67.1, R7.1, R77.1
- net I2C_LED_SCL: now also U10.22 (SCL)
- net I2C_LED_SDA: now also U10.23 (SDA)
- net at R100.2: now also U10.1 (~{INT})
- net at R14.2, U2.2 (-): now also R15.1; no longer R15.2
- net at R66.2, U7.3 (+): now also R67.1; no longer R67.2
- net at R46.2, U5.3 (+): now also R47.1; no longer R47.2
- net at R34.2, U4.2 (-): now also R35.1; no longer R35.2
- net at R54.2, U6.2 (-): now also R55.1; no longer R55.2
- net at R24.2, U3.2 (-): now also R25.1; no longer R25.2
- net at R74.2, U8.2 (-): now also R75.1; no longer R75.2
- net at R76.2, U8.3 (+): now also R77.1; no longer R77.2
- net at R44.2, U5.2 (-): now also R45.1; no longer R45.2
- net at U11.2 (ALERT_RDY): now also R101.1; no longer R101.2
- net at R4.2, U1.2 (-): now also R5.1; no longer R5.2
- net at R56.2, U6.3 (+): now also R57.1; no longer R57.2
- net at R6.2, U1.3 (+): now also R7.1; no longer R7.2
- net at R26.2, U3.3 (+): now also R27.1; no longer R27.2
- net at R16.2, U2.3 (+): now also R17.1; no longer R17.2
- net at R64.2, U7.2 (-): now also R65.1; no longer R65.2
- net at R36.2, U4.3 (+): now also R37.1; no longer R37.2
- net at U12.2 (ALERT_RDY): now also R102.1; no longer R102.2
- new net: R65.2, R68.1, U7.1
- new net: R35.2, R38.1, U4.1
- new net: R75.2, R78.1, U8.1
- new net: R25.2, R28.1, U3.1
- new net: R5.2, R8.1, U1.1
- new net: R45.2, R48.1, U5.1
- new net: R15.2, R18.1, U2.1
- new net: R55.2, R58.1, U6.1
- no-connect marks 0 -> 32
