File: Hardware (kicad)/MPCBoard/MPCBoard.kicad_pcb (KiCad board)
At the start: 2 copper layers, 145 x 95 mm, 118 parts, among them J1 62000421821, J2 62000421821, J3 62000421821, J4 62000421821, J5 62000421821, J6 62000421821, J7 62000421821, J8 62000421821, P1 61300611121, U1 TS914, U10 PCA9535A, U11 ADS1015IDGST, U12 ADS1015IDGST, U2 TS914, U3 TS914, U4 TS914, U5 TS914, U6 TS914, U7 TS914, U8 TS914

Commit message: fix kicad projects
Parts:
- C1, C100, C101, C102, C11, C12, C2, C21, C22, C31, C32, C41, C42, C51, C52, C61, C62, C71, C72: footprint Passive SMD:CAPC0603(1608)100_N -> Capacitor_SMD:C_0603_1608Metric_Pad1.08x0.95mm_HandSolder
- R1, R100, R101, R102, R103, R104, R105, R106, R11, R12, R13, R14, R15, R16, R17, R18, R2, R21, R22, R23, R24, R25, R26, R27, R28, R3, R31, R32, R33, R34, R35, R36, R37, R38, R4, R41, R42, R43, R44, R45, R46, R47, R48, R5, R51, R52, R53, R54, R55, R56, R57, R58, R6, R61, R62, R63, R64, R65, R66, R67, R68, R7, R71, R72, R73, R74, R75, R76, R77, R78, R8: footprint Passive SMD:RESC0603(1608)_N -> Resistor_SMD:R_0603_1608Metric_Pad0.98x0.95mm_HandSolder
- U1, U2, U3, U4, U5, U6, U7, U8: footprint TS914AIDT:SO-14_STM -> Sampler:TS914IDT
- U11, U12: footprint ADS1015IDGST:DGS0010A_N -> ADS1015IDGST:SOP50P490X110-10N
- moved R103 1.54 mm to (96.7, 61.4)
- moved R106 0.94 mm to (85.2, 61.4)
- moved R3 0.80 mm to (89.4, 97.4)
- moved R104 0.34 mm to (92.7, 61.4)
- moved R105 0.28 mm to (89.0, 61.4)
- moved C1 0.21 mm to (102.5, 95.2), turned to 0 degrees
- moved R56 0.21 mm to (173.1, 123.8)
- moved R46 0.21 mm to (173.2, 88.5)
- turned R102 to 90 degrees
- turned C11 to 0 degrees
- turned C21 to 0 degrees
- turned C31 to 0 degrees
- turned C41 to 0 degrees
- turned C51 to 0 degrees
- turned C61 to 0 degrees
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Connections:
- net NetJ1_2 renamed LED_01
- net NetJ2_2 renamed LED_02
- net NetJ3_2 renamed LED_03
- net NetJ4_2 renamed LED_04
- net NetJ5_2 renamed LED_05
- net NetJ6_2 renamed LED_06
- net NetJ7_2 renamed LED_07
- net NetJ8_2 renamed LED_08
- net NetP1_3 renamed I2C_LED_SCL
- net NetP1_4 renamed I2C_LED_SDA
- net NetP1_5 renamed I2C_BTN_SCL
- net NetP1_6 renamed I2C_BTN_SDA
- net NetR100_2 renamed Net-(U10A-~{INT})
- net NetR12_2 renamed BTN_02-
- net NetR14_1 renamed Net-(U2C--)
- net NetR16_1 renamed Net-(U2D--)
- net NetR22_2 renamed BTN_03-
- net NetR24_1 renamed Net-(U3C--)
- net NetR26_1 renamed Net-(U3D--)
- net NetR2_2 renamed BTN_01-
- net NetR32_2 renamed BTN_04-
- net NetR34_1 renamed Net-(U4C--)
- net NetR36_1 renamed Net-(U4D--)
- net NetR42_2 renamed BTN_05-
- net NetR44_1 renamed Net-(U5C--)
- net NetR46_1 renamed Net-(U5D--)
- net NetR4_1 renamed Net-(U1C--)
- net NetR52_2 renamed BTN_06-
- net NetR54_1 renamed Net-(U6C--)
- net NetR56_1 renamed Net-(U6D--)
- net NetR62_2 renamed BTN_07-
- net NetR64_1 renamed Net-(U7C--)
- net NetR66_1 renamed Net-(U7D--)
- net NetR6_1 renamed Net-(U1D--)
- net NetR72_2 renamed BTN_08-
- net NetR74_1 renamed Net-(U8C--)
- net NetR76_1 renamed Net-(U8D--)
- C1 pad 1: GND -> BTN_01+
- C1 pad 2: NetC1_2 -> GND
- C11 pad 1: GND -> BTN_02+
- C11 pad 2: NetC11_2 -> GND
- C21 pad 1: GND -> BTN_03+
- C21 pad 2: NetC21_2 -> GND
- C31 pad 1: GND -> BTN_04+
- C31 pad 2: NetC31_2 -> GND
- C41 pad 1: GND -> BTN_05+
- C41 pad 2: NetC41_2 -> GND
- C51 pad 1: GND -> BTN_06+
- C51 pad 2: NetC51_2 -> GND
- C61 pad 1: GND -> BTN_07+
- C61 pad 2: NetC61_2 -> GND
- C71 pad 1: GND -> BTN_08+
- C71 pad 2: NetC71_2 -> GND
- J1 pad 3: NetC1_2 -> BTN_01+
- J2 pad 3: NetC11_2 -> BTN_02+
- J3 pad 3: NetC21_2 -> BTN_03+
- J4 pad 3: NetC31_2 -> BTN_04+
- J5 pad 3: NetC41_2 -> BTN_05+
- J6 pad 3: NetC51_2 -> BTN_06+
- J7 pad 3: NetC61_2 -> BTN_07+
- J8 pad 3: NetC71_2 -> BTN_08+
- R1 pad 1: NetC1_2 -> BTN_01+
- R101 pad 1: +5V -> Net-(U11-ALERT_RDY)
- R101 pad 2: NetR101_2 -> +5V
- R102 pad 1: +5V -> Net-(U12-ALERT_RDY)
- R102 pad 2: NetR102_2 -> +5V
- R11 pad 1: NetC11_2 -> BTN_02+
- R14 pad 2: NetR14_2 -> Net-(U2A--)
- R15 pad 1: NetR15_1 -> Net-(U2A--)
- R15 pad 2: NetR14_2 -> Net-(R15-Pad2)
- R16 pad 2: NetR16_2 -> Net-(U2A-+)
- R17 pad 1: GND -> Net-(U2A-+)
- R17 pad 2: NetR16_2 -> GND
- R18 pad 1: NetR18_1 -> Net-(R15-Pad2)
- R18 pad 2: NetR15_1 -> BTN_02_OUT
- R21 pad 1: NetC21_2 -> BTN_03+
- R24 pad 2: NetR24_2 -> Net-(U3A--)
- R25 pad 1: NetR25_1 -> Net-(U3A--)
- R25 pad 2: NetR24_2 -> Net-(R25-Pad2)
- R26 pad 2: NetR26_2 -> Net-(U3A-+)
- R27 pad 1: GND -> Net-(U3A-+)
- R27 pad 2: NetR26_2 -> GND
- R28 pad 1: NetR28_1 -> Net-(R25-Pad2)
- R28 pad 2: NetR25_1 -> BTN_03_OUT
- R31 pad 1: NetC31_2 -> BTN_04+
- R34 pad 2: NetR34_2 -> Net-(U4A--)
- R35 pad 1: NetR35_1 -> Net-(U4A--)
- R35 pad 2: NetR34_2 -> Net-(R35-Pad2)
- R36 pad 2: NetR36_2 -> Net-(U4A-+)
- R37 pad 1: GND -> Net-(U4A-+)
- R37 pad 2: NetR36_2 -> GND
- R38 pad 1: NetR38_1 -> Net-(R35-Pad2)
- R38 pad 2: NetR35_1 -> BTN_04_OUT
- R4 pad 2: NetR4_2 -> Net-(U1A--)
- R41 pad 1: NetC41_2 -> BTN_05+
- R44 pad 2: NetR44_2 -> Net-(U5A--)
- R45 pad 1: NetR45_1 -> Net-(U5A--)
- R45 pad 2: NetR44_2 -> Net-(R45-Pad2)
- R46 pad 2: NetR46_2 -> Net-(U5A-+)
- R47 pad 1: GND -> Net-(U5A-+)
- R47 pad 2: NetR46_2 -> GND
- R48 pad 1: NetR48_1 -> Net-(R45-Pad2)
- R48 pad 2: NetR45_1 -> BTN_05_OUT
- R5 pad 1: NetR5_1 -> Net-(U1A--)
- R5 pad 2: NetR4_2 -> Net-(R5-Pad2)
- R51 pad 1: NetC51_2 -> BTN_06+
- R54 pad 2: NetR54_2 -> Net-(U6A--)
- R55 pad 1: NetR55_1 -> Net-(U6A--)
- R55 pad 2: NetR54_2 -> Net-(R55-Pad2)
- R56 pad 2: NetR56_2 -> Net-(U6A-+)
- R57 pad 1: GND -> Net-(U6A-+)
- R57 pad 2: NetR56_2 -> GND
- R58 pad 1: NetR58_1 -> Net-(R55-Pad2)
- R58 pad 2: NetR55_1 -> BTN_06_OUT
- R6 pad 2: NetR6_2 -> Net-(U1A-+)
- R61 pad 1: NetC61_2 -> BTN_07+
- R64 pad 2: NetR64_2 -> Net-(U7A--)
- R65 pad 1: NetR65_1 -> Net-(U7A--)
- R65 pad 2: NetR64_2 -> Net-(R65-Pad2)
- R66 pad 2: NetR66_2 -> Net-(U7A-+)
- R67 pad 1: GND -> Net-(U7A-+)
- R67 pad 2: NetR66_2 -> GND
- R68 pad 1: NetR68_1 -> Net-(R65-Pad2)
- R68 pad 2: NetR65_1 -> BTN_07_OUT
- R7 pad 1: GND -> Net-(U1A-+)
- R7 pad 2: NetR6_2 -> GND
- R71 pad 1: NetC71_2 -> BTN_08+
- R74 pad 2: NetR74_2 -> Net-(U8A--)
- R75 pad 1: NetR75_1 -> Net-(U8A--)
- R75 pad 2: NetR74_2 -> Net-(R75-Pad2)
- R76 pad 2: NetR76_2 -> Net-(U8A-+)
- R77 pad 1: GND -> Net-(U8A-+)
- R77 pad 2: NetR76_2 -> GND
- R78 pad 1: NetR78_1 -> Net-(R75-Pad2)
- R78 pad 2: NetR75_1 -> BTN_08_OUT
- R8 pad 1: NetR8_1 -> Net-(R5-Pad2)
- R8 pad 2: NetR5_1 -> BTN_01_OUT
- U1 pad 1: NetR5_1 -> Net-(R5-Pad2)
- U1 pad 12: NetC1_2 -> BTN_01+
- U1 pad 2: NetR4_2 -> Net-(U1A--)
- U1 pad 3: NetR6_2 -> Net-(U1A-+)
- U1 pad 5: (no net) -> unconnected-(U1B-+-Pad5)
- U1 pad 6: (no net) -> unconnected-(U1B---Pad6)
- U1 pad 7: (no net) -> unconnected-(U1-Pad7)
- U10 pad 13: (no net) -> unconnected-(U10C-P1_0-Pad13)
- U10 pad 14: (no net) -> unconnected-(U10C-P1_1-Pad14)
- U10 pad 15: (no net) -> unconnected-(U10C-P1_2-Pad15)
- U10 pad 16: (no net) -> unconnected-(U10C-P1_3-Pad16)
- U10 pad 17: (no net) -> unconnected-(U10C-P1_4-Pad17)
- U10 pad 18: (no net) -> unconnected-(U10C-P1_5-Pad18)
- U10 pad 19: (no net) -> unconnected-(U10C-P1_6-Pad19)
- U10 pad 20: (no net) -> unconnected-(U10C-P1_7-Pad20)
- U11 pad 2: NetR101_2 -> Net-(U11-ALERT_RDY)
- U11 pad 4: NetR8_1 -> BTN_01_OUT
- U11 pad 5: NetR18_1 -> BTN_02_OUT
- U11 pad 6: NetR28_1 -> BTN_03_OUT
- U11 pad 7: NetR38_1 -> BTN_04_OUT
- U12 pad 2: NetR102_2 -> Net-(U12-ALERT_RDY)
- U12 pad 4: NetR48_1 -> BTN_05_OUT
- U12 pad 5: NetR58_1 -> BTN_06_OUT
- U12 pad 6: NetR68_1 -> BTN_07_OUT
- U12 pad 7: NetR78_1 -> BTN_08_OUT
- U2 pad 1: NetR15_1 -> Net-(R15-Pad2)
- U2 pad 12: NetC11_2 -> BTN_02+
- U2 pad 2: NetR14_2 -> Net-(U2A--)
- U2 pad 3: NetR16_2 -> Net-(U2A-+)
- U2 pad 5: (no net) -> unconnected-(U2B-+-Pad5)
- U2 pad 6: (no net) -> unconnected-(U2B---Pad6)
- U2 pad 7: (no net) -> unconnected-(U2-Pad7)
- U3 pad 1: NetR25_1 -> Net-(R25-Pad2)
- U3 pad 12: NetC21_2 -> BTN_03+
- U3 pad 2: NetR24_2 -> Net-(U3A--)
- U3 pad 3: NetR26_2 -> Net-(U3A-+)
- U3 pad 5: (no net) -> unconnected-(U3B-+-Pad5)
- U3 pad 6: (no net) -> unconnected-(U3B---Pad6)
- U3 pad 7: (no net) -> unconnected-(U3-Pad7)
- U4 pad 1: NetR35_1 -> Net-(R35-Pad2)
- U4 pad 12: NetC31_2 -> BTN_04+
- U4 pad 2: NetR34_2 -> Net-(U4A--)
- U4 pad 3: NetR36_2 -> Net-(U4A-+)
- U4 pad 5: (no net) -> unconnected-(U4B-+-Pad5)
- U4 pad 6: (no net) -> unconnected-(U4B---Pad6)
- U4 pad 7: (no net) -> unconnected-(U4-Pad7)
- U5 pad 1: NetR45_1 -> Net-(R45-Pad2)
- U5 pad 12: NetC41_2 -> BTN_05+
- U5 pad 2: NetR44_2 -> Net-(U5A--)
- U5 pad 3: NetR46_2 -> Net-(U5A-+)
- U5 pad 5: (no net) -> unconnected-(U5B-+-Pad5)
- U5 pad 6: (no net) -> unconnected-(U5B---Pad6)
- U5 pad 7: (no net) -> unconnected-(U5-Pad7)
- U6 pad 1: NetR55_1 -> Net-(R55-Pad2)
- U6 pad 12: NetC51_2 -> BTN_06+
- U6 pad 2: NetR54_2 -> Net-(U6A--)
- U6 pad 3: NetR56_2 -> Net-(U6A-+)
- U6 pad 5: (no net) -> unconnected-(U6B-+-Pad5)
- U6 pad 6: (no net) -> unconnected-(U6B---Pad6)
- U6 pad 7: (no net) -> unconnected-(U6-Pad7)
- U7 pad 1: NetR65_1 -> Net-(R65-Pad2)
- U7 pad 12: NetC61_2 -> BTN_07+
- U7 pad 2: NetR64_2 -> Net-(U7A--)
- U7 pad 3: NetR66_2 -> Net-(U7A-+)
- U7 pad 5: (no net) -> unconnected-(U7B-+-Pad5)
- U7 pad 6: (no net) -> unconnected-(U7B---Pad6)
- U7 pad 7: (no net) -> unconnected-(U7-Pad7)
- U8 pad 1: NetR75_1 -> Net-(R75-Pad2)
- U8 pad 12: NetC71_2 -> BTN_08+
- U8 pad 2: NetR74_2 -> Net-(U8A--)
- U8 pad 3: NetR76_2 -> Net-(U8A-+)
- U8 pad 5: (no net) -> unconnected-(U8B-+-Pad5)
- U8 pad 6: (no net) -> unconnected-(U8B---Pad6)
- U8 pad 7: (no net) -> unconnected-(U8-Pad7)
Routing:
- net NetR38_1: track 78.6 -> 0.00 mm, vias 2 -> 0
- net BTN_04_OUT: track 0.00 -> 78.6 mm, vias 0 -> 2
- net NetR78_1: track 76.8 -> 0.00 mm, vias 2 -> 0
- net BTN_08_OUT: track 0.00 -> 76.8 mm, vias 0 -> 2
- net NetR58_1: track 47.3 -> 0.00 mm, vias 2 -> 0
- net BTN_06_OUT: track 0.00 -> 47.3 mm, vias 0 -> 2
- net NetR18_1: track 46.5 -> 0.00 mm, vias 2 -> 0
- net BTN_02_OUT: track 0.00 -> 46.5 mm, vias 0 -> 2
- net NetR28_1: track 45.0 -> 0.00 mm
- net BTN_03_OUT: track 0.00 -> 45.0 mm
- net NetR68_1: track 43.4 -> 0.00 mm
- net BTN_07_OUT: track 0.00 -> 43.4 mm
- net NetR54_2: track 18.5 -> 0.00 mm
- net Net-(U6A--): track 0.00 -> 18.5 mm
- net NetR14_2: track 18.3 -> 0.00 mm
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Other:
- rule pad_to_mask_clearance: 0.1016 -> 0.075
